File: Business Card v2.kicad_pcb (KiCad board)
At the start: 2 copper layers, 85.4 x 54.1 mm, 39 parts, among them J1 Conn_01x03_Pin, Q1 DMP21D0UFB4-P, U1 ATTINY816-MNR, U3 NT3H2111W0FHKH

Commit message: Updates
Parts:
- C1: value 1.5pF -> 1.5p
- C2, C4: value 100nF -> 100n
- C3: value 10uF -> 10u
- LED22: value (none) -> XL-1608UYC-06FJ
Connections:
- net Net-(U1-PB0) renamed /INDICATOR_LED
Changed lines of the file:
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@@
 	(net 27 "/UPDI_PAD")
 	(net 28 "/GATE")
-	(net 29 "Net-(U1-PB0)")
+	(net 29 "/INDICATOR_LED")
 	(net 30 "Net-(LED22-A)")
 	(net 31 "unconnected-(U1-PC1-Pad16)")
@@
 			)
 		)
-		(property "Value" "100nF"
+		(property "Value" "100n"
 			(at 0 1.16 45)
 			(layer "F.Fab")
@@
 			(size 0.2 0.8)
 			(layers "F.Cu" "F.Mask" "F.Paste")
-			(net 29 "Net-(U1-PB0)")
+			(net 29 "/INDICATOR_LED")
 			(pinfunction "PB0")
 			(pintype "unspecified")
@@
 			)
 		)
-		(property "Value" "100nF"
+		(property "Value" "100n"
 			(at 0 1.16 0)
 			(layer "F.Fab")
@@
 			)
 		)
-		(property "Value" ""
+		(property "Value" "XL-1608UYC-06FJ"
 			(at 0 1.745846 90)
 			(layer "F.Fab")
@@
 			)
 		)
-		(property "Datasheet" ""
+		(property "Datasheet" "https://wmsc.lcsc.com/wmsc/upload/file/pdf/v2/lcsc/2402181501_XINGLIGHT-XL-1608UYC-06FJ_C7371901.pdf"
 			(at 0 0 90)
 			(layer "F.Fab")
@@
 			)
 		)
-		(property "Description" ""
+		(property "Description" "-40℃~+85℃ 1.6mm x 0.8mm square LED 1.9V~2.3V 120° 20mA 587nm~595nm 590nm 600mcd 60mW Discrete Diode Top-mount Water Clear Yellow 0603 LED Indication - Discrete ROHS"
 			(at 0 0 90)
 			(layer "F.Fab")
@@
 			)
 		)
-		(property "LCSC" "C7371900"
+		(property "LCSC" "C7371901"
 			(at 0 0 90)
 			(layer "F.Fab")
@@
 			)
 		)
-		(property "Manufacturer Part" ""
+		(property "Manufacturer Part" "XL-1608UYC-06FJ"
 			(at 0 0 270)
 			(unlocked yes)
@@
 			)
 		)
-		(property "Value" "10uF"
+		(property "Value" "10u"
 			(at 0 1.16 0)
 			(layer "F.Fab")
@@
 			(layers "F.Cu" "F.Mask" "F.Paste")
 			(roundrect_rratio 0.25)
-			(net 29 "Net-(U1-PB0)")
+			(net 29 "/INDICATOR_LED")
 			(pintype "passive")
 		)
@@
 			)
 		)
-		(property "Value" "1.5pF"
+		(property "Value" "1.5p"
 			(at 0 1.16 180)
 			(layer "F.Fab")
