File: Business Card v2.kicad_sch (KiCad schematic)
At the start: 39 parts, among them J1 Conn_01x03_Pin, Q1 DMP21D0UFB4-P, U1 ATTINY816-MNR, U3 NT3H2111W0FHKH

Commit message: Updates
Parts:
- C1: value 1.5pF -> 1.5p
- C2, C4: value 100nF -> 100n
- C3: value 10uF -> 10u
Changed lines of the file:
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@@
 			)
 		)
-		(property "Value" "100nF"
+		(property "Value" "100n"
 			(at 67.31 80.0099 0)
 			(effects
@@
 			)
 		)
-		(property "Value" "1.5pF"
+		(property "Value" "1.5p"
 			(at 53.34 50.7999 0)
 			(effects
@@
 			)
 		)
-		(property "Value" "10uF"
+		(property "Value" "10u"
 			(at 137.16 77.4699 0)
 			(effects
@@
 			)
 		)
-		(property "Value" "100nF"
+		(property "Value" "100n"
 			(at 195.58 60.9599 0)
 			(effects
